File: power_mosfet.kicad_sch (KiCad schematic)
At the start: 14 parts, among them Q1 Q_NMOS, Q2 Q_NMOS, Q3 Q_NMOS, Q4 Q_NMOS, Q5 Q_NMOS, Q6 Q_NMOS

Commit message: MOSFET part number updated
Parts:
- Q1, Q2, Q3, Q4, Q5, Q6: value Q_NMOS -> IPD25N06S4L30ATM
Changed lines of the file:
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@@
 			)
 		)
-		(property "Value" "Q_NMOS"
+		(property "Value" "IPD25N06S4L30ATM"
 			(at 142.24 85.0899 0)
 			(show_name no)
@@
 			)
 		)
-		(property "Value" "Q_NMOS"
+		(property "Value" "IPD25N06S4L30ATM"
 			(at 82.55 58.4199 0)
 			(show_name no)
@@
 			)
 		)
-		(property "Value" "Q_NMOS"
+		(property "Value" "IPD25N06S4L30ATM"
 			(at 142.24 58.4199 0)
 			(show_name no)
@@
 			)
 		)
-		(property "Value" "Q_NMOS"
+		(property "Value" "IPD25N06S4L30ATM"
 			(at 219.71 58.4199 0)
 			(show_name no)
@@
 			)
 		)
-		(property "Value" "Q_NMOS"
+		(property "Value" "IPD25N06S4L30ATM"
 			(at 82.55 85.0899 0)
 			(show_name no)
@@
 			)
 		)
-		(property "Value" "Q_NMOS"
+		(property "Value" "IPD25N06S4L30ATM"
 			(at 219.71 85.0899 0)
 			(show_name no)
